File: Controller Board/Controller Board.kicad_sch (KiCad schematic)
At the start: 19 parts, among them J1 Conn_01x03, J2 Fan_connector, K1 G3MB-202PDC5 Relay, SW1 SW_SPDT, U1 attiny85, U2 AMS1117-5.0, U3 AMS1117-5.0

Commit message: updated schematic
Parts:
- removed C2: 10uF, Capacitor_SMD:C_0805_2012Metric_Pad1.18x1.45mm_HandSolder, symbol Device:C
- removed C3: 22uF, Capacitor_SMD:C_0805_2012Metric_Pad1.18x1.45mm_HandSolder, symbol Device:C
- removed U2: AMS1117-5.0, Package_TO_SOT_SMD:SOT-223-3_TabPin2, symbol Regulator_Linear:AMS1117-5.0
- added D2: D, 000_Thomas_Footprints:Diode-SOD-80, symbol Device:D
- added J2: Conn_01x04, Connector_PinHeader_2.54mm:PinHeader_1x04_P2.54mm_Vertical, symbol Connector_Generic:Conn_01x04
- H1, H2: footprint MountingHole:MountingHole_2.2mm_M2 -> MountingHole:MountingHole_3.2mm_M3
- renumbered C4 to C1, C5 to C2, D2 to D3, J2 to J1, J1 to J3, U3 to U2
Connections:
- net Vcc: now also SW1.2 (B)
- net Vin: no longer SW1.2 (B)
- net MISO: now reaches R2.1, U1.6 (PB1)
- net MISO: now also J2.3 (Pin_3)
- net MOSI: now reaches U1.5 (PB0)
- net MOSI: now also J2.4 (Pin_4); no longer R1.2
- net Reset: now reaches RST1.2, U1.1 (PB5)
- net Reset: now also J2.1 (Pin_1)
- net trigger: now reaches U1.2 (PB3)
- net trigger: now also R1.2, SW1.1 (A), D2.1 (K)
- net SCK: now reaches U1.7 (PB2)
- net SCK: now also J2.2 (Pin_2)
- net trigger_pin: no longer names the net of J3.3 (Pin_3)
- net trigger_pin: now also D2.2 (A); no longer SW1.3 (C)
- no-connect marks 3 -> 1
Other:
- note added: "Programming Pins"
- note removed: "Voltage Reader"
- moved on the sheet: D1, J3, R2, RST1, SW1
