File: Controller Board/Controller Board.kicad_sch (KiCad schematic)
At the start: 18 parts, among them J1 Fan_connector, J2 Conn_01x04, J3 Conn_01x03, K1 G3MB-202PDC5 Relay, SW1 SW_SPDT, U1 attiny85, U2 AMS1117-5.0

Commit message: final version
Parts:
- removed K1: G3MB-202PDC5 Relay, 000_Thomas_Footprints:G3MB-202PDC5 Relay, symbol 000_Thomas_Symbols:G3MB-202PDC5 Relay
- removed U1: attiny85, Package_DIP:DIP-8_W7.62mm, symbol 000_Thomas_Symbols:ATTINY85
- added K1: AQG22105, 0_Thomas_Footprints:RELAY_AQG22105, symbol 0_Thomas_Symbols:AQG22105 Relay
- added U1: attiny85, Package_DIP:DIP-8_W7.62mm, symbol 0_Thomas_Symbols:ATTINY85
- D2: footprint 000_Thomas_Footprints:Diode-SOD-80 -> 0_Thomas_Footprints:Diode-SOD-80
- J1: footprint 000_Thomas_Footprints:myTerminalBlock-2_P5.08mm -> 0_Thomas_Footprints:myTerminalBlock-2_P5.08mm
- RST1: footprint 000_Thomas_Footprints:SW_PTS636_SM43J_SMTR_LFS -> 0_Thomas_Footprints:SW_PTS636_SM43J_SMTR_LFS
- SW1: footprint 000_Thomas_Footprints:EG1218 Slide Switch -> 0_Thomas_Footprints:EG1218 Slide Switch
Connections:
- net GND: now also K1.4 (Sig-), U1.4 (GND)
- net MISO: now also U1.6 (PB1)
- net MOSI: now also U1.5 (PB0)
- net Reset: now also U1.1 (PB5)
- net SCK: now also U1.7 (PB2)
- net Vcc: now also U1.8 (Vcc)
- net trigger: now also U1.2 (PB3)
- net at J1.1 (Pin_1): now also K1.1 (OUT1)
- net at J1.2 (Pin_2): now also K1.2 (OUT2)
- new net: K1.3 (Sig+), U1.3 (PB4)
