File: Controller Board/Controller Board.kicad_pcb (KiCad board)
At the start: 2 copper layers, 50.3 x 25.9 mm, 18 parts, among them J1 Fan_connector, J2 Conn_01x04, J3 Conn_01x03, K1 G3MB-202PDC5 Relay, SW1 SW_SPDT, U1 attiny85, U2 AMS1117-5.0

Commit message: final version
Parts:
- D2: footprint 000_Thomas_Footprints:Diode-SOD-80 -> 0_Thomas_Footprints:Diode-SOD-80
- J1: footprint 000_Thomas_Footprints:myTerminalBlock-2_P5.08mm -> 0_Thomas_Footprints:myTerminalBlock-2_P5.08mm
- K1: value G3MB-202PDC5 Relay -> AQG22105; footprint 000_Thomas_Footprints:G3MB-202PDC5 Relay -> 0_Thomas_Footprints:RELAY_AQG22105
- RST1: footprint 000_Thomas_Footprints:SW_PTS636_SM43J_SMTR_LFS -> 0_Thomas_Footprints:SW_PTS636_SM43J_SMTR_LFS
- SW1: footprint 000_Thomas_Footprints:EG1218 Slide Switch -> 0_Thomas_Footprints:EG1218 Slide Switch
- moved K1 2.20 mm to (143.3, 90.4)
